File: PCB/macro.kicad_sch (KiCad schematic)
At the start: 39 parts, among them SW1 SW_Push, SW10 SW_Push, SW11 SW_Push, SW12 SW_Push, SW13 SW_Push, SW14 SW_Push, SW15 SW_Push, SW16 SW_Push, SW17 SW_Push, SW2 SW_Push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

Commit message: Rev3v3 in production
Parts:
- added D18, D19: Red Diode 1206, symbol Device:LED_Filled
- added Dr1k, Dy1k: 1kΩ, symbol PCM_Elektuur:R
- D1, D10, D11, D12, D13, D14, D15, D16, D17, D2, D3, D4, D5, D6, D7, D8, D9: value 1N4148WT -> 1206
Connections:
- net at Arduino.31 (PC6), SW5.1, SW6.1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: now also Arduino.9 (PB1), D19.2 (A)
- net at Arduino.15 (GND), Arduino.23 (GND), Arduino.35 (GND)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: now also Dr1k.2 (-), Dy1k.2 (-)
- net at Arduino.10 (PB2): now also D18.2 (A)
- new net: D18.1 (K), Dy1k.1 (+)
- new net: D19.1 (K), Dr1k.1 (+)
Other:
- moved on the sheet: Arduino, Cl1, Cl2, Cl3, Cl4, D1, D10, D11, D12, D13, D14, D15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
