File: PCB/macro=REV2.kicad_pcb (KiCad board)
At the start: 2 copper layers, 102 x 110 mm, 52 parts

Commit message: REV3 almost done
Parts:
- added ?: , , F.Cu at (94.9, 101.8)
- added ?: , , F.Cu at (117.9, 122.6)
- added ?: , , F.Cu at (87.5, 122.3)
- added ?: , , F.Cu at (138.4, 112.0)
- added ?: , , F.Cu at (85.0, 122.3)
- added ?: , , F.Cu at (97.5, 101.8)
- added ?: , , F.Cu at (115.4, 122.6)
- added ?: , , F.Cu at (135.9, 112.0)
- moved ? 9.73 mm to (136.1, 71.9)
- moved ? 9.73 mm to (138.7, 71.9)
- moved ? 8.89 mm to (138.4, 40.8)
- moved ? 8.89 mm to (135.9, 40.8)
- moved ? 8.76 mm to (118.0, 81.3)
- moved ? 8.76 mm to (115.4, 81.3)
- moved ? 8.66 mm to (115.3, 40.5)
- moved ? 8.66 mm to (117.9, 40.5)
- moved ? 8.58 mm to (115.3, 60.8)
- moved ? 8.58 mm to (117.8, 60.8)
- moved ? 8.33 mm to (117.5, 101.5)
- moved ? 8.33 mm to (115.0, 101.5)
- moved ? 8.23 mm to (94.6, 81.3)
- moved ? 8.23 mm to (97.1, 81.3)
- moved ? 8.10 mm to (97.0, 40.6)
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Routing:
- net (no net): track 140.6 -> 1618.3 mm, vias 0 -> 6

Commit message: Rev3v3 in production
Parts:
- removed ? (x42): , 
- added 1kR1: R_1206_3216Metric, PCM_Resistor_SMD_AKL:R_1206_3216Metric, F.Cu at (65.2, 119.0)
- added 1kR2: R_1206_3216Metric, PCM_Resistor_SMD_AKL:R_1206_3216Metric, F.Cu at (69.2, 119.0)
- added 1kR3: R_1206_3216Metric, PCM_Resistor_SMD_AKL:R_1206_3216Metric, B.Cu at (149.5, 34.8)
- added 1kR4: R_1206_3216Metric, PCM_Resistor_SMD_AKL:R_1206_3216Metric, B.Cu at (149.5, 40.0)
- added 1kR5: R_1206_3216Metric, PCM_Resistor_SMD_AKL:R_1206_3216Metric, B.Cu at (149.5, 47.5)
- added 1kR6: R_1206_3216Metric, PCM_Resistor_SMD_AKL:R_1206_3216Metric, B.Cu at (149.5, 50.0)
- added D1: D_1206_3216Metric_Pad1.42x1.75mm_HandSolder, PCM_Diode_SMD_AKL:D_1206_3216Metric_Pad1.42x1.75mm_HandSolder, F.Cu at (81.2, 25.2)
- added D10: D_1206_3216Metric_Pad1.42x1.75mm_HandSolder, PCM_Diode_SMD_AKL:D_1206_3216Metric_Pad1.42x1.75mm_HandSolder, F.Cu at (121.8, 65.8)
- added D11: D_1206_3216Metric_Pad1.42x1.75mm_HandSolder, PCM_Diode_SMD_AKL:D_1206_3216Metric_Pad1.42x1.75mm_HandSolder, F.Cu at (139.5, 81.2)
- added D12: D_1206_3216Metric_Pad1.42x1.75mm_HandSolder, PCM_Diode_SMD_AKL:D_1206_3216Metric_Pad1.42x1.75mm_HandSolder, F.Cu at (81.2, 86.2)
- added D13: D_1206_3216Metric_Pad1.42x1.75mm_HandSolder, PCM_Diode_SMD_AKL:D_1206_3216Metric_Pad1.42x1.75mm_HandSolder, F.Cu at (101.5, 86.2)
- added D14: D_1206_3216Metric_Pad1.42x1.75mm_HandSolder, PCM_Diode_SMD_AKL:D_1206_3216Metric_Pad1.42x1.75mm_HandSolder, F.Cu at (121.8, 86.5)
- added D15: D_1206_3216Metric_Pad1.42x1.75mm_HandSolder, PCM_Diode_SMD_AKL:D_1206_3216Metric_Pad1.42x1.75mm_HandSolder, F.Cu at (91.8, 106.5)
- added D16: D_1206_3216Metric_Pad1.42x1.75mm_HandSolder, PCM_Diode_SMD_AKL:D_1206_3216Metric_Pad1.42x1.75mm_HandSolder, F.Cu at (121.8, 106.5)
- added D17: D_1206_3216Metric_Pad1.42x1.75mm_HandSolder, PCM_Diode_SMD_AKL:D_1206_3216Metric_Pad1.42x1.75mm_HandSolder, F.Cu at (139.8, 110.8)
- added D2: D_1206_3216Metric_Pad1.42x1.75mm_HandSolder, PCM_Diode_SMD_AKL:D_1206_3216Metric_Pad1.42x1.75mm_HandSolder, F.Cu at (101.5, 25.2)
- added D3: D_1206_3216Metric_Pad1.42x1.75mm_HandSolder, PCM_Diode_SMD_AKL:D_1206_3216Metric_Pad1.42x1.75mm_HandSolder, F.Cu at (121.8, 25.0)
- added D4: D_1206_3216Metric_Pad1.42x1.75mm_HandSolder, PCM_Diode_SMD_AKL:D_1206_3216Metric_Pad1.42x1.75mm_HandSolder, F.Cu at (139.5, 40.8)
- added D5: D_1206_3216Metric_Pad1.42x1.75mm_HandSolder, PCM_Diode_SMD_AKL:D_1206_3216Metric_Pad1.42x1.75mm_HandSolder, F.Cu at (81.2, 45.8)
- added D6: D_1206_3216Metric_Pad1.42x1.75mm_HandSolder, PCM_Diode_SMD_AKL:D_1206_3216Metric_Pad1.42x1.75mm_HandSolder, F.Cu at (101.5, 45.8)
- added D7: D_1206_3216Metric_Pad1.42x1.75mm_HandSolder, PCM_Diode_SMD_AKL:D_1206_3216Metric_Pad1.42x1.75mm_HandSolder, F.Cu at (121.8, 45.2)
- added D8: D_1206_3216Metric_Pad1.42x1.75mm_HandSolder, PCM_Diode_SMD_AKL:D_1206_3216Metric_Pad1.42x1.75mm_HandSolder, F.Cu at (81.2, 66.0)
- added D9: D_1206_3216Metric_Pad1.42x1.75mm_HandSolder, PCM_Diode_SMD_AKL:D_1206_3216Metric_Pad1.42x1.75mm_HandSolder, F.Cu at (101.5, 65.8)
- added LED18: D_1210_3225Metric_Pad1.42x2.65mm_HandSolder, PCM_Diode_SMD_AKL:D_1210_3225Metric_Pad1.42x2.65mm_HandSolder, F.Cu at (145.8, 127.0)
- added LED19: D_1210_3225Metric_Pad1.42x2.65mm_HandSolder, PCM_Diode_SMD_AKL:D_1210_3225Metric_Pad1.42x2.65mm_HandSolder, F.Cu at (152.0, 127.0)
Routing:
- net (no net): track 1618.3 -> 1980.6 mm, vias 6 -> 2
Other:
- board text removed: "Cl1 1kΩ"
- board text removed: "Cl2 1kΩ"
- board text removed: "Cl3 1kΩ"
- board text removed: "Cl4 1kΩ"
- board text removed: "Diode"
